Commit message: minor fixes

File: romnibot/chefbot_description/urdf/chefbot_base.urdf.xacro (robot description, xacro)
@@ -7,6 +7,6 @@
  -->
 <robot name="chefbot" xmlns:xacro="http://ros.org/wiki/xacro">
-  <xacro:include filename="$(find romni_description)/urdf/common_properties.urdf.xacro"/>
-  <xacro:include filename="$(find romni_description)/urdf/chefbot_base_gazebo.urdf.xacro"/>
+  <xacro:include filename="$(find chefbot_description)/urdf/common_properties.urdf.xacro"/>
+  <xacro:include filename="$(find chefbot_description)/urdf/chefbot_base_gazebo.urdf.xacro"/>
   <!-- Chefbot -->
   <xacro:macro name="kobuki">
@@ -30,5 +30,5 @@
         <geometry>
           <!-- new mesh -->
-          <mesh filename="package://romni_description/meshes/base_plate.dae" />
+          <mesh filename="package://chefbot_description/meshes/base_plate.dae" />
         </geometry>
 <!--        <origin xyz="0.001 0 0.05199" rpy="0 0 ${M_PI/2}"/> -->
@@ -66,5 +66,5 @@
       <visual>
         <geometry>
-          <mesh filename="package://romni_description/meshes/wheel.dae"/>
+          <mesh filename="package://chefbot_description/meshes/wheel.dae"/>
         </geometry>
         <origin xyz="0 0 0" rpy="0 0 0"/>
@@ -93,5 +93,5 @@
       <visual>
         <geometry>
-          <mesh filename="package://romni_description/meshes/wheel.dae"/>
+          <mesh filename="package://chefbot_description/meshes/wheel.dae"/>
         </geometry>
         <origin xyz="0 0 0" rpy="0 0 0"/>
